File: odonata_split/PCB_Files/odonata_split.kicad_pcb (KiCad board)
At the start: 2 copper layers, 134.2 x 96 mm, 56 parts, among them J1 trrs_num, K1 KEYSW, K10 KEYSW, K11 KEYSW, K12 KEYSW, K13 KEYSW, K14 KEYSW, K15 KEYSW, K16 KEYSW, K17 KEYSW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

Commit message: begin naming refactor
Parts:
- added G***: LOGO, logo:odonata_logo_text3, B.Cu at (214.4, 69.8)
- added G***: LOGO, logo:odonata_logo_text3, F.Cu at (214.4, 83.5)
